Commit message: Fix arm dimensions

File: src/chessmate_description/urdf/scara_robot.urdf.xacro (robot description, xacro)
@@ -5,4 +5,6 @@
   <xacro:property name="link1_length" value="0.202" />
   <xacro:property name="link2_length" value="0.190" />
+  <xacro:property name="link1_width" value="0.044" />
+  <xacro:property name="link2_width" value="0.022" />
   <xacro:property name="base_height" value="0.1" />
   <!-- Base Link -->
@@ -39,5 +41,5 @@
       <origin xyz="${link1_length/2} 0 0" rpy="0 0 0"/>
       <geometry>
-        <box size="${link1_length} 0.05 0.05"/>
+        <box size="${link1_length} ${link1_width} ${link1_width}"/>
       </geometry>
       <material name="link_color">
@@ -48,5 +50,5 @@
       <origin xyz="${link1_length/2} 0 0" rpy="0 0 0"/>
       <geometry>
-        <box size="${link1_length} 0.05 0.05"/>
+        <box size="${link1_length} ${link1_width} ${link1_width}"/>
       </geometry>
     </collision>
@@ -70,5 +72,5 @@
       <origin xyz="${link2_length/2} 0 0" rpy="0 0 0"/>
       <geometry>
-        <box size="${link2_length} 0.04 0.04"/>
+        <box size="${link2_length} ${link2_width} ${link2_width}"/>
       </geometry>
       <material name="link_color">
@@ -79,5 +81,5 @@
       <origin xyz="${link2_length/2} 0 0" rpy="0 0 0"/>
       <geometry>
-        <box size="${link2_length} 0.04 0.04"/>
+        <box size="${link2_length} ${link2_width} ${link2_width}"/>
       </geometry>
     </collision>
@@ -94,5 +96,5 @@
     <origin xyz="${link2_length} 0 0" rpy="0 0 0"/>
     <axis xyz="0 0 1"/>
-    <limit lower="0" upper="0.05" effort="5" velocity="0.1"/>
+    <limit lower="0" upper="0.1" effort="5" velocity="0.1"/>
   </joint>
   <!-- End Effector -->

Commit message: fix z movement

File: src/chessmate_description/urdf/scara_robot.urdf.xacro (robot description, xacro)
@@ -28,9 +28,37 @@
     </inertial>
   </link>
+  <!-- Z-axis joint (vertical base movement) -->
+  <joint name="z_joint" type="prismatic">
+    <parent link="base_link"/>
+    <child link="z_carriage"/>
+    <origin xyz="0 0 ${base_height/2}" rpy="0 0 0"/>
+    <axis xyz="0 0 1"/>
+    <limit lower="0" upper="0.1" effort="5" velocity="0.1"/>
+  </joint>
+  <!-- Z-axis carriage (moves vertically) -->
+  <link name="z_carriage">
+    <visual>
+      <geometry>
+        <cylinder radius="0.03" length="0.02"/>
+      </geometry>
+      <material name="carriage_color">
+        <color rgba="0.6 0.6 0.6 1.0"/>
+      </material>
+    </visual>
+    <collision>
+      <geometry>
+        <cylinder radius="0.03" length="0.02"/>
+      </geometry>
+    </collision>
+    <inertial>
+      <mass value="0.2"/>
+      <inertia ixx="0.0001" ixy="0" ixz="0" iyy="0.0001" iyz="0" izz="0.0001"/>
+    </inertial>
+  </link>
   <!-- Joint 1 (Base rotation) -->
   <joint name="base_joint" type="revolute">
-    <parent link="base_link"/>
+    <parent link="z_carriage"/>
     <child link="link1"/>
-    <origin xyz="0 0 ${base_height/2}" rpy="0 0 0"/>
+    <origin xyz="0 0 0" rpy="0 0 0"/>
     <axis xyz="0 0 1"/>
     <limit lower="-1.57" upper="1.57" effort="10" velocity="2.0"/>
@@ -90,11 +118,9 @@
     </inertial>
   </link>
-  <!-- Z-axis joint (vertical) -->
-  <joint name="z_joint" type="prismatic">
+  <!-- End Effector Joint -->
+  <joint name="end_effector_joint" type="fixed">
     <parent link="link2"/>
     <child link="end_effector"/>
     <origin xyz="${link2_length} 0 0" rpy="0 0 0"/>
-    <axis xyz="0 0 1"/>
-    <limit lower="0" upper="0.1" effort="5" velocity="0.1"/>
   </joint>
   <!-- End Effector -->

Commit message: Reflect the mechanical linkage between L1 and L2

File: src/chessmate_description/urdf/scara_robot.urdf.xacro (robot description, xacro)
@@ -87,9 +87,25 @@
     </inertial>
   </link>
-  <!-- Joint 2 (Shoulder) -->
+  <!-- Intermediate link for mechanical coupling -->
+  <joint name="coupling_joint" type="revolute">
+    <parent link="link1"/>
+    <child link="coupling_link"/>
+    <origin xyz="${link1_length} 0 0" rpy="0 0 0"/>
+    <axis xyz="0 0 1"/>
+    <limit lower="-3.14" upper="3.14" effort="10" velocity="2.0"/>
+    <mimic joint="base_joint" multiplier="-1.0" offset="0.0"/>
+  </joint>
+  <!-- Coupling link (invisible, just for kinematics) -->
+  <link name="coupling_link">
+    <inertial>
+      <mass value="0.001"/>
+      <inertia ixx="0.00001" ixy="0" ixz="0" iyy="0.00001" iyz="0" izz="0.00001"/>
+    </inertial>
+  </link>
+  <!-- Joint 2 (Independent L2 control) -->
   <joint name="shoulder_joint" type="revolute">
-    <parent link="link1"/>
+    <parent link="coupling_link"/>
     <child link="link2"/>
-    <origin xyz="${link1_length} 0 0" rpy="0 0 0"/>
+    <origin xyz="0 0 0" rpy="0 0 0"/>
     <axis xyz="0 0 1"/>
     <limit lower="-1.57" upper="1.57" effort="10" velocity="2.0"/>

Commit message: Upload meshes

File: src/chessmate_description/urdf/scara_robot.urdf.xacro (robot description, xacro)
@@ -8,10 +8,21 @@
   <xacro:property name="link2_width" value="0.022" />
   <xacro:property name="base_height" value="0.1" />
+  <!-- Mesh usage flag - set to true when STL files are available -->
+  <xacro:property name="use_meshes" value="true" />
+  <!-- Package path for meshes -->
+  <xacro:property name="mesh_path" value="package://chessmate_description/meshes" />
   <!-- Base Link -->
   <link name="base_link">
     <visual>
-      <geometry>
-        <cylinder radius="0.05" length="${base_height}"/>
-      </geometry>
+      <xacro:if value="${use_meshes}">
+        <geometry>
+          <mesh filename="${mesh_path}/visual/base_link_visual.stl" scale="0.001 0.001 0.001"/>
+        </geometry>
+      </xacro:if>
+      <xacro:unless value="${use_meshes}">
+        <geometry>
+          <cylinder radius="0.05" length="${base_height}"/>
+        </geometry>
+      </xacro:unless>
       <material name="base_color">
         <color rgba="0.5 0.5 0.5 1.0"/>
@@ -19,7 +30,14 @@
     </visual>
     <collision>
-      <geometry>
-        <cylinder radius="0.05" length="${base_height}"/>
-      </geometry>
+      <xacro:if value="${use_meshes}">
+        <geometry>
+          <mesh filename="${mesh_path}/collision/base_link_collision.stl" scale="0.001 0.001 0.001"/>
+        </geometry>
+      </xacro:if>
+      <xacro:unless value="${use_meshes}">
+        <geometry>
+          <cylinder radius="0.05" length="${base_height}"/>
+        </geometry>
+      </xacro:unless>
     </collision>
     <inertial>
@@ -67,17 +85,32 @@
   <link name="link1">
     <visual>
-      <origin xyz="${link1_length/2} 0 0" rpy="0 0 0"/>
-      <geometry>
-        <box size="${link1_length} ${link1_width} ${link1_width}"/>
-      </geometry>
-      <material name="link_color">
+      <xacro:if value="${use_meshes}">
+        <origin xyz="0 0 0" rpy="0 0 0"/>
+        <geometry>
+          <mesh filename="${mesh_path}/visual/link1_visual.stl" scale="0.001 0.001 0.001"/>
+        </geometry>
+      </xacro:if>
+      <xacro:unless value="${use_meshes}">
+        <origin xyz="${link1_length/2} 0 0" rpy="0 0 0"/>
+        <geometry>
+          <box size="${link1_length} ${link1_width} ${link1_width}"/>
+        </geometry>
+      </xacro:unless>
+      <material name="link1_color">
         <color rgba="0.8 0.2 0.2 1.0"/>
       </material>
     </visual>
     <collision>
-      <origin xyz="${link1_length/2} 0 0" rpy="0 0 0"/>
-      <geometry>
-        <box size="${link1_length} ${link1_width} ${link1_width}"/>
-      </geometry>
+      <xacro:if value="${use_meshes}">
+        <geometry>
+          <mesh filename="${mesh_path}/collision/link1_collision.stl" scale="0.001 0.001 0.001"/>
+        </geometry>
+      </xacro:if>
+      <xacro:unless value="${use_meshes}">
+        <origin xyz="${link1_length/2} 0 0" rpy="0 0 0"/>
+        <geometry>
+          <box size="${link1_length} ${link1_width} ${link1_width}"/>
+        </geometry>
+      </xacro:unless>
     </collision>
     <inertial>
@@ -114,17 +147,32 @@
   <link name="link2">
     <visual>
-      <origin xyz="${link2_length/2} 0 0" rpy="0 0 0"/>
-      <geometry>
-        <box size="${link2_length} ${link2_width} ${link2_width}"/>
-      </geometry>
-      <material name="link_color">
+      <xacro:if value="${use_meshes}">
+        <origin xyz="0 0 0" rpy="0 0 0"/>
+        <geometry>
+          <mesh filename="${mesh_path}/visual/link2_visual.stl" scale="0.001 0.001 0.001"/>
+        </geometry>
+      </xacro:if>
+      <xacro:unless value="${use_meshes}">
+        <origin xyz="${link2_length/2} 0 0" rpy="0 0 0"/>
+        <geometry>
+          <box size="${link2_length} ${link2_width} ${link2_width}"/>
+        </geometry>
+      </xacro:unless>
+      <material name="link2_color">
         <color rgba="0.2 0.8 0.2 1.0"/>
       </material>
     </visual>
     <collision>
-      <origin xyz="${link2_length/2} 0 0" rpy="0 0 0"/>
-      <geometry>
-        <box size="${link2_length} ${link2_width} ${link2_width}"/>
-      </geometry>
+      <xacro:if value="${use_meshes}">
+        <geometry>
+          <mesh filename="${mesh_path}/collision/link2_collision.stl" scale="0.001 0.001 0.001"/>
+        </geometry>
+      </xacro:if>
+      <xacro:unless value="${use_meshes}">
+        <origin xyz="${link2_length/2} 0 0" rpy="0 0 0"/>
+        <geometry>
+          <box size="${link2_length} ${link2_width} ${link2_width}"/>
+        </geometry>
+      </xacro:unless>
     </collision>
     <inertial>
@@ -143,7 +191,14 @@
   <link name="end_effector">
     <visual>
-      <geometry>
-        <box size="0.03 0.03 0.02"/>
-      </geometry>
+      <xacro:if value="${use_meshes}">
+        <geometry>
+          <mesh filename="${mesh_path}/visual/end_effector_visual.stl" scale="0.001 0.001 0.001"/>
+        </geometry>
+      </xacro:if>
+      <xacro:unless value="${use_meshes}">
+        <geometry>
+          <box size="0.03 0.03 0.02"/>
+        </geometry>
+      </xacro:unless>
       <material name="gripper_color">
         <color rgba="0.2 0.2 0.8 1.0"/>
@@ -151,7 +206,14 @@
     </visual>
     <collision>
-      <geometry>
-        <box size="0.03 0.03 0.02"/>
-      </geometry>
+      <xacro:if value="${use_meshes}">
+        <geometry>
+          <mesh filename="${mesh_path}/collision/end_effector_collision.stl" scale="0.001 0.001 0.001"/>
+        </geometry>
+      </xacro:if>
+      <xacro:unless value="${use_meshes}">
+        <geometry>
+          <box size="0.03 0.03 0.02"/>
+        </geometry>
+      </xacro:unless>
     </collision>
     <inertial>

Commit message: adjust the origins for the arm to look its part

File: src/chessmate_description/urdf/scara_robot.urdf.xacro (robot description, xacro)
@@ -12,8 +12,17 @@
   <!-- Package path for meshes -->
   <xacro:property name="mesh_path" value="package://chessmate_description/meshes" />
+  <!-- World frame (root of the robot) -->
+  <link name="world"/>
+  <!-- Joint to position base_link in world coordinate system -->
+  <joint name="world_to_base" type="fixed">
+    <parent link="world"/>
+    <child link="base_link"/>
+    <origin xyz="0 0 0" rpy="0 0 0"/>
+  </joint>
   <!-- Base Link -->
   <link name="base_link">
     <visual>
       <xacro:if value="${use_meshes}">
+        <origin xyz="-0.05 0 -0.1" rpy="1.5708 0 1.5708"/>
         <geometry>
           <mesh filename="${mesh_path}/visual/base_link_visual.stl" scale="0.001 0.001 0.001"/>
@@ -31,4 +40,5 @@
     <collision>
       <xacro:if value="${use_meshes}">
+        <origin xyz="0 0 -0.1" rpy="1.5708 0 0"/>
         <geometry>
           <mesh filename="${mesh_path}/collision/base_link_collision.stl" scale="0.001 0.001 0.001"/>
@@ -86,5 +96,5 @@
     <visual>
       <xacro:if value="${use_meshes}">
-        <origin xyz="0 0 0" rpy="0 0 0"/>
+        <origin xyz="0.05 0 0" rpy="1.57 0 -1.57"/>
         <geometry>
           <mesh filename="${mesh_path}/visual/link1_visual.stl" scale="0.001 0.001 0.001"/>
@@ -148,5 +158,5 @@
     <visual>
       <xacro:if value="${use_meshes}">
-        <origin xyz="0 0 0" rpy="0 0 0"/>
+        <origin xyz="-0.075 -0.025 0.01" rpy="0 0 -3.14159"/>
         <geometry>
           <mesh filename="${mesh_path}/visual/link2_visual.stl" scale="0.001 0.001 0.001"/>
@@ -192,4 +202,5 @@
     <visual>
       <xacro:if value="${use_meshes}">
+        <origin xyz="-0.035 -0.015 0" rpy="0 0 0"/>
         <geometry>
           <mesh filename="${mesh_path}/visual/end_effector_visual.stl" scale="0.001 0.001 0.001"/>

Commit message: Add collision avoidance

File: src/chessmate_description/urdf/scara_robot.urdf.xacro (robot description, xacro)
@@ -147,4 +147,5 @@
   </link>
   <!-- Joint 2 (Independent L2 control) -->
+  <!-- Limits set to prevent self-collision: 30° buffer on each side -->
   <joint name="shoulder_joint" type="revolute">
     <parent link="coupling_link"/>
@@ -152,5 +153,6 @@
     <origin xyz="0 0 0" rpy="0 0 0"/>
     <axis xyz="0 0 1"/>
-    <limit lower="-1.57" upper="1.57" effort="10" velocity="2.0"/>
+    <limit lower="-2.618" upper="2.618" effort="10" velocity="2.0"/>
+    <!-- lower=-150°, upper=+150° to maintain 30° buffer from ±180° folded position -->
   </joint>
   <!-- Link 2 -->
